Commit message: lidar cad

File: wc_robot/config/wc.urdf (robot description, URDF)
Before this commit: robot wc_robot, 6 links, 5 joints
Joints:
- joint base_left_wheel_joint: axis 0 1 0 -> 0 0 1
- joint base_right_wheel_joint: axis 0 1 0 -> 0 0 1

File: wc_robot/config/wc.urdf.xacro (robot description, xacro)
@@ -100,4 +100,29 @@
         </plugin>
     </gazebo>
+    <gazebo>
+        <plugin name="gazebo_ros_joint_state_publisher" filename="libgazebo_ros_joint_state_publisher.so">
+            <update_rate>20</update_rate>
+            <joint_name>base_joint</joint_name>
+            <joint_name>base_lidar_joint</joint_name>
+            <joint_name>base_left_wheel_joint</joint_name>
+            <joint_name>base_right_wheel_joint</joint_name>
+            <joint_name>base_castor</joint_name>
+        </plugin>
+    </gazebo>
+    <gazebo reference="base_link">
+        <material>Gazebo/Green</material>
+    </gazebo>
+    <gazebo reference="lidar">
+        <material>Gazebo/White</material>
+    </gazebo>
+    <gazebo reference="left_wheel">
+        <material>Gazebo/Grey</material>
+    </gazebo>
+    <gazebo reference="right_wheel">
+        <material>Gazebo/Grey</material>
+    </gazebo>
+    <gazebo reference="castor_wheel">
+        <material>Gazebo/Grey</material>
+    </gazebo>
 <!-- LIDAR Sensor -->
     <gazebo reference="lidar">
