Commit message: Update wc_bot.urdf

File: wc_ws/src/wc_description/urdf/wc_bot.urdf (robot description, URDF)
Before this commit: robot wc_bot, 8 links, 7 joints
Links:
- link base_link: geometry collision box size=0.510 0.510 0.094; visual mesh filename=package://wc_description/meshes/bases/wc_base.stl scale=0.001 0.001 0.001
